Commit message: xacro+collisions

File: urdf/bobik_robot.urdf (robot description, URDF)
Before this commit: robot bobik, 8 links, 7 joints
Links:
- added link lidar_link, mass 0.2; collision box size=0.08 0.08 0.045; visual cylinder length=0.018 radius=0.04
- link base_link: geometry collision mesh filename=file:///home/honza/ros2_foxy/src/bobik_robot/meshes/base_li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; visual mesh filename=file:///home/honza/ros2_foxy/src/bobik_robot/meshes/base_li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
- link fl_caster_wheel_link: geometry collision box size=0.123 0.024 0.123; visual cylinder length=0.024 radius=0.0615
- link fr_caster_wheel_link: geometry collision box size=0.123 0.024 0.123; visual cylinder length=0.024 radius=0.0615
- link r_caster_wheel_link: geometry collision box size=0.123 0.024 0.123; visual cylinder length=0.024 radius=0.0615
Joints:
- added joint lidar_joint: type fixed, parent base_link, child lidar_link
- joint fl_caster_rotation_joint: origin xyz=0.224 0.23 0.08 rpy=0 0 0.0 -> xyz=0.134 0.23 0.173 rpy=0 0 0.0
- joint fl_caster_wheel_joint: origin xyz=0 0 0 rpy=0 0 0 -> xyz=0 0 -0.110 rpy=0 0 0
- joint fr_caster_rotation_joint: origin xyz=0.224 -0.23 0.08 rpy=0 0 0.0 -> xyz=0.134 -0.23 0.173 rpy=0 0 0.0
- joint fr_caster_wheel_joint: origin xyz=0 0 0 rpy=0 0 0 -> xyz=0 0 -0.110 rpy=0 0 0
- joint r_caster_rotation_joint: origin xyz=-0.18 0.0 0.08 rpy=0 0 0.0 -> xyz=-0.270 0.0 0.173 rpy=0 0 0.0
- joint r_caster_wheel_joint: origin xyz=0 0 0 rpy=0 0 0 -> xyz=0 0 -0.110 rpy=0 0 0

File: urdf/bobik_robot.urdf.xacro (robot description, xacro)
@@ -21,5 +21,5 @@
             <origin xyz="0 0 0" rpy="0 0 0" />
             <geometry>
-                <box size="0.5 0.5 0.2" />
+                <mesh filename="file:///home/honza/ros2_foxy/src/bobik_robot/meshes/base_link_collision.dae" />
             </geometry>
         </collision>
@@ -40,5 +40,5 @@
         <link name="${prefix}_caster_rotation_link">
             <visual>
-                <origin xyz="-0.04 -0.024 -0.025" rpy="0 0 0" />
+                <origin xyz="0 0 0" rpy="0 0 0" />
                 <geometry>
                     <mesh filename="package://bobik_robot/meshes/caster_rotation_link.dae" />
@@ -46,11 +46,11 @@
             </visual>
             <collision>
-                <origin xyz="0 0.013 0.029" rpy="0 0 0" />
+                <origin xyz="0 0 -0.06" rpy="0 0 0" />
                 <geometry>
-                    <box size="0.08 0.075 0.11" />
+                    <box size="0.10 0.11 0.12" />
                 </geometry>
             </collision>
             <inertial>
-                <origin xyz="-0.04 -0.026 -0.025" rpy="0 0 0" />
+                <origin xyz="0 0 -0.1" rpy="0 0 0" />
                 <mass value="0.5" />
                 <inertia ixx="2.2124416e-03" ixy="-1.2294101e-05" ixz="3.4938785e-05" iyy="2.1193702e-03" iyz="-5.0120904e-06" izz="2.0064271e-03" />
@@ -60,5 +60,5 @@
             <parent link="${prefix}_caster_rotation_link" />
             <child link="${prefix}_caster_wheel_link" />
-            <origin xyz="0 0 0" rpy="0 0 0" />
+            <origin xyz="0 0 -0.110" rpy="0 0 0" />
             <axis xyz="0 1 0" />
             <limit effort="30" velocity="${M_PI*2}" />
@@ -85,6 +85,30 @@
         </link>
     </xacro:macro>
-    <xacro:caster prefix="fl" joint_origin="0.224 0.23 0.08" />
-    <xacro:caster prefix="fr" joint_origin="0.224 -0.23 0.08" />
-    <xacro:caster prefix="r"  joint_origin="-0.18 0.0 0.08" />
+    <xacro:caster prefix="fl" joint_origin="0.134 0.23 0.173" />
+    <xacro:caster prefix="fr" joint_origin="0.134 -0.23 0.173" />
+    <xacro:caster prefix="r"  joint_origin="-0.270 0.0 0.173" />
+    <joint name="lidar_joint" type="fixed">
+        <parent link="base_link" />
+        <child link="lidar_link" />
+        <origin xyz="0.12 0.13 ${0.045/2+0.21}" rpy="0 0 0" />
+    </joint>
+    <link name="lidar_link">
+        <visual>
+            <origin xyz="0 0 0" rpy="0 0 0" />
+            <geometry>
+                <cylinder length="0.018" radius="0.04" />
+            </geometry>
+            <material name="black"/>
+        </visual>
+        <collision>
+            <origin xyz="0 0 0" rpy="0 0 0" />
+            <geometry>
+                <box size="0.08 0.08 0.045" />
+            </geometry>
+        </collision>
+        <inertial>
+            <origin xyz="0 0 0" rpy="0 0 0" />
+            <mass value="0.2" />
+            <inertia ixx="2.2124416e-04" ixy="-1.2294101e-06" ixz="3.4938785e-06" iyy="2.1193702e-04" iyz="-5.0120904e-05" izz="2.0064271e-04" />        </inertial>
+    </link>
 </robot>

Commit message: ekf setup

File: urdf/bobik_robot.urdf (robot description, URDF)
Before this commit: robot bobik, 9 links, 8 joints
Links:
- removed link base_footprint
- link fl_caster_rotation_link: geometry collision box size=0.10 0.11 0.12; visual mesh filename=package://bobik_robot/meshes/caster_rotation_link.dae
- link fr_caster_rotation_link: geometry collision box size=0.10 0.11 0.12; visual mesh filename=package://bobik_robot/meshes/caster_rotation_link.dae
- link r_caster_rotation_link: geometry collision box size=0.10 0.11 0.12; visual mesh filename=package://bobik_robot/meshes/caster_rotation_link.dae
Joints:
- removed joint root_joint
- joint lidar_joint: origin (none) -> xyz=0.12 0.13 0.23249999999999998 rpy=0 0 0

File: urdf/bobik_robot.urdf.xacro (robot description, xacro)
@@ -6,9 +6,9 @@
     <xacro:property name="wheel_diameter" value="0.123" />
     <!-- root_link is a workaround for base_link to have an inertia mass -->
-    <link name="base_footprint"></link>
+    <!-- <link name="base_footprint"></link>
     <joint name="root_joint" type="fixed">
         <parent link="base_footprint" />
         <child link="base_link" />
-    </joint>
+    </joint> -->
     <link name="base_link">
         <visual>
