Commit message: human request

File: urdf/bobik_robot.urdf.xacro (robot description, xacro)
@@ -24,9 +24,9 @@
             </geometry>
         </collision>
-        <inertial>
+        <!--<inertial>
             <origin xyz="0 0 0" rpy="0 0 0" />
             <mass value="1.5" />
             <inertia ixx="2.2124416e-03" ixy="-1.2294101e-05" ixz="3.4938785e-05" iyy="2.1193702e-03" iyz="-5.0120904e-06" izz="2.0064271e-03" />
-        </inertial>
+        </inertial>-->
     </link>
     <xacro:macro name="caster" params="prefix joint_origin">

Commit message: adding imu, draft

File: urdf/bobik_robot.urdf.xacro (robot description, xacro)
@@ -110,5 +110,31 @@
             <origin xyz="0 0 0" rpy="0 0 0" />
             <mass value="0.2" />
-            <inertia ixx="2.2124416e-04" ixy="-1.2294101e-06" ixz="3.4938785e-06" iyy="2.1193702e-04" iyz="-5.0120904e-05" izz="2.0064271e-04" />        </inertial>
+            <inertia ixx="2.2124416e-04" ixy="-1.2294101e-06" ixz="3.4938785e-06" iyy="2.1193702e-04" iyz="-5.0120904e-05" izz="2.0064271e-04" />
+        </inertial>
+    </link>
+    <joint name="imu_joint" type="fixed">
+        <parent link="base_link" />
+        <child link="imu_link" />
+        <origin xyz="-0.1 0.0 0.16" rpy="0 0 0" />
+    </joint>
+    <link name="imu_link">
+        <visual>
+            <origin xyz="0 0 0" rpy="0 0 0" />
+            <geometry>
+                <box size="0.016 0.02 0.01" />
+            </geometry>
+            <material name="blue"/>
+        </visual>
+        <collision>
+            <origin xyz="0 0 0" rpy="0 0 0" />
+            <geometry>
+                <box size="0.016 0.02 0.01" />
+            </geometry>
+        </collision>
+        <inertial>
+            <origin xyz="0 0 0" rpy="0 0 0" />
+            <mass value="0.01" />
+            <inertia ixx="2.2124416e-04" ixy="-1.2294101e-06" ixz="3.4938785e-06" iyy="2.1193702e-04" iyz="-5.0120904e-05" izz="2.0064271e-04" />
+        </inertial>
     </link>
 </robot>
